Commit message: [feat] checkpoint: functional autonomous line following

File: iot/software/src/speedy_description/urdf/speedy.urdf.xacro (robot description, xacro)
@@ -6,198 +6,261 @@
   <xacro:arg name="hardware_config_file" default="" />
   <xacro:property name="hw_config_path" value="$(arg hardware_config_file)" />
-  <!-- Carrega parâmetros do hardware.yaml se o arquivo for fornecido -->
   <xacro:if value="${hw_config_path != ''}">
     <xacro:property name="hw_config" value="${xacro.load_yaml(hw_config_path)['speedy_hardware']['ros__parameters']}" />
-    <!-- Converte graus para radianos pro URDF -->
-    <xacro:property name="max_steer_angle_left" value="${hw_config['max_steering_angle_left_deg'] * (pi / 180.0)}" />
+    <xacro:property name="max_steer_angle_left"  value="${hw_config['max_steering_angle_left_deg']  * (pi / 180.0)}" />
     <xacro:property name="max_steer_angle_right" value="${hw_config['max_steering_angle_right_deg'] * (pi / 180.0)}" />
+    <xacro:property name="wheelbase"    value="${hw_config['wheelbase']}" />
+    <xacro:property name="wheel_radius" value="${hw_config['wheel_radius']}" />
   </xacro:if>
   <xacro:unless value="${hw_config_path != ''}">
-    <xacro:property name="max_steer_angle_left" value="0.785398" />
+    <xacro:property name="max_steer_angle_left"  value="0.785398" />
     <xacro:property name="max_steer_angle_right" value="0.785398" />
+    <xacro:property name="wheelbase"    value="0.251" />
+    <xacro:property name="wheel_radius" value="0.0325" />
+    <xacro:property name="hw_config" value="${dict()}" />
   </xacro:unless>
-  <!-- Dimensões Físicas -->
-  <xacro:property name="chassis_length" value="0.252" />
-  <xacro:property name="chassis_width"  value="0.166" />
-  <xacro:property name="chassis_height" value="0.0755" />
-  <xacro:property name="bumper_length" value="0.057" />
-  <xacro:property name="bumper_width"  value="0.137" />
-  <xacro:property name="bumper_height" value="0.044" />
-  <xacro:property name="wheel_radius" value="0.0325" />
-  <xacro:property name="wheel_width"  value="0.026" />
-  <xacro:property name="wheelbase"    value="0.251" />
-  <xacro:property name="track_width"  value="0.139" />
-  <xacro:property name="chassis_z_offset" value="0.017" />
-  <!-- Materiais Visuais -->
-  <material name="white">
-    <color rgba="0.9 0.9 0.9 1.0"/>
-  </material>
-  <material name="blue">
-    <color rgba="0.1 0.3 0.8 1.0"/>
-  </material>
-  <material name="black">
-    <color rgba="0.15 0.15 0.15 1.0"/>
-  </material>
-  <!-- ============================================== -->
-  <!-- DESCRIÇÃO CINEMÁTICA E VISUAL                  -->
-  <!-- ============================================== -->
-  <!-- Chassi Base -->
-  <link name="base_link">
-    <visual>
-      <origin xyz="-0.006 0 ${chassis_z_offset + (chassis_height/2)}" rpy="0 0 0"/>
-      <geometry>
-        <box size="${chassis_length} ${chassis_width} ${chassis_height}"/>
-      </geometry>
-      <material name="white"/>
-    </visual>
-    <collision>
-      <origin xyz="-0.006 0 ${chassis_z_offset + (chassis_height/2)}" rpy="0 0 0"/>
-      <geometry>
-        <box size="${chassis_length} ${chassis_width} ${chassis_height}"/>
-      </geometry>
-    </collision>
-  </link>
-  <!-- Para-choque Dianteiro -->
-  <link name="front_bumper_link">
-    <visual>
-      <origin xyz="${(chassis_length/2) + (bumper_length/2) - 0.006} 0 ${chassis_z_offset + (bumper_height/2)}" rpy="0 0 0"/>
-      <geometry>
-        <box size="${bumper_length} ${bumper_width} ${bumper_height}"/>
-      </geometry>
-      <material name="blue"/>
-    </visual>
-  </link>
-  <joint name="front_bumper_joint" type="fixed">
-    <parent link="base_link"/>
-    <child link="front_bumper_link"/>
-  </joint>
-  <!-- Para-choque Traseiro -->
-  <link name="rear_bumper_link">
-    <visual>
-      <origin xyz="${-(chassis_length/2) - (bumper_length/2) - 0.006} 0 ${chassis_z_offset + (bumper_height/2)}" rpy="0 0 0"/>
-      <geometry>
-        <box size="${bumper_length} ${bumper_width} ${bumper_height}"/>
-      </geometry>
-      <material name="blue"/>
-    </visual>
-  </link>
-  <joint name="rear_bumper_joint" type="fixed">
-    <parent link="base_link"/>
-    <child link="rear_bumper_link"/>
-  </joint>
-  <!-- Sensor IMU MPU6050 -->
-  <link name="imu_link">
-    <visual>
-      <origin xyz="0 0 0" rpy="0 0 0"/>
-      <geometry>
-        <box size="0.020 0.015 0.002"/>
-      </geometry>
-      <material name="black"/>
-    </visual>
-  </link>
-  <!-- Pinos para a esquerda: Rotação em Z (yaw) pode precisar de ajuste dependendo de como a placa mapeia X/Y -->
-  <joint name="imu_joint" type="fixed">
-    <parent link="base_link"/>
-    <child link="imu_link"/>
-    <origin xyz="0 0 ${chassis_z_offset + chassis_height}" rpy="0 0 0"/>
-  </joint>
-  <!-- Juntas Virtuais (Reais pro ros2_control) -->
+  <!-- ============================================== -->
+  <!-- DIMENSÕES FÍSICAS (metros)                     -->
+  <!--   Fonte: medições físicas do chassi            -->
+  <!--   wheelbase e wheel_radius: hardware.yaml      -->
+  <!-- ============================================== -->
+  <!-- Chassi principal -->
+  <xacro:property name="chassis_length"   value="0.259"  />  <!-- 38.5 total - 2*6.3 bumper = 25.9 -->
+  <xacro:property name="chassis_height"   value="0.080"  />  <!-- medido pelo usuário -->
+  <xacro:property name="chassis_width"    value="0.166"  />
+  <!-- Caixa do LiDAR no topo do chassi -->
+  <xacro:property name="lidar_box_l"       value="0.130" />
+  <xacro:property name="lidar_box_w"       value="0.090" />
+  <xacro:property name="lidar_box_h"       value="0.065" />
+  <!-- Rodas -->
+  <xacro:property name="wheel_thickness"  value="0.026"  />
+  <!-- distância do centro do chassi ao centro da roda (eixo Y) -->
+  <xacro:property name="half_track"       value="0.0695" />
+  <!-- quanto a roda projeta para cima, acima do topo do chassi -->
+  <xacro:property name="wheel_projection" value="0.020"  />
+  <!-- Pára-choques -->
+  <xacro:property name="bumper_length"    value="0.063"  />  <!-- medido pelo usuário -->
+  <xacro:property name="bumper_height"    value="0.050"  />  <!-- medido pelo usuário -->
+  <xacro:property name="bumper_width"     value="0.137"  />
+  <!-- Distância do eixo da roda até a extremidade do pára-choque (medido: 6.5cm) -->
+  <xacro:property name="wheel_to_bumper_edge" value="0.065" />
+  <!-- ============================================== -->
+  <!-- DESCRIÇÃO CINEMÁTICA                           -->
+  <!-- ============================================== -->
+  <!-- base_link na altura do eixo das rodas, no ponto médio entre eixos -->
+  <link name="base_link" />
+  <!-- Eixo traseiro (tração) -->
   <link name="drive_wheel_link" />
   <joint name="drive_joint" type="continuous">
     <parent link="base_link"/>
     <child link="drive_wheel_link"/>
-    <origin xyz="${-wheelbase/2} 0 0" rpy="0 0 0"/>
+    <!-- Centraliza visualmente o wheelbase no chassi -->
+    <origin xyz="${-wheelbase/2.0} 0 0" rpy="0 0 0"/>
     <axis xyz="0 1 0"/>
   </joint>
+  <!-- Eixo dianteiro (direção) -->
   <link name="steering_link" />
   <joint name="steering_joint" type="revolute">
     <parent link="base_link"/>
     <child link="steering_link"/>
-    <origin xyz="${wheelbase/2} 0 0" rpy="0 0 0"/>
+    <origin xyz="${wheelbase/2.0} 0 0" rpy="0 0 0"/>
     <axis xyz="0 0 1"/>
     <limit lower="${-max_steer_angle_right}" upper="${max_steer_angle_left}" effort="10.0" velocity="5.0"/>
   </joint>
-  <!-- Rodas Físicas Visuais (Mimics) -->
-  <link name="rl_wheel_link">
-    <visual>
-      <origin xyz="0 0 0" rpy="${pi/2} 0 0"/>
-      <geometry>
-        <cylinder radius="${wheel_radius}" length="${wheel_width}"/>
-      </geometry>
-      <material name="black"/>
-    </visual>
-  </link>
-  <joint name="rl_wheel_joint" type="continuous">
-    <parent link="base_link"/>
-    <child link="rl_wheel_link"/>
-    <origin xyz="${-wheelbase/2} ${track_width/2} 0" rpy="0 0 0"/>
-    <axis xyz="0 1 0"/>
-    <mimic joint="drive_joint" multiplier="1.0" offset="0.0"/>
-  </joint>
-  <link name="rr_wheel_link">
-    <visual>
-      <origin xyz="0 0 0" rpy="${pi/2} 0 0"/>
-      <geometry>
-        <cylinder radius="${wheel_radius}" length="${wheel_width}"/>
-      </geometry>
-      <material name="black"/>
-    </visual>
-  </link>
-  <joint name="rr_wheel_joint" type="continuous">
-    <parent link="base_link"/>
-    <child link="rr_wheel_link"/>
-    <origin xyz="${-wheelbase/2} ${-track_width/2} 0" rpy="0 0 0"/>
-    <axis xyz="0 1 0"/>
-    <mimic joint="drive_joint" multiplier="1.0" offset="0.0"/>
-  </joint>
-  <link name="fl_steer_link" />
-  <joint name="fl_steer_joint" type="revolute">
-    <parent link="base_link"/>
-    <child link="fl_steer_link"/>
-    <origin xyz="${wheelbase/2} ${track_width/2} 0" rpy="0 0 0"/>
+  <!-- ============================================== -->
+  <!-- GEOMETRIA VISUAL E DE COLISÃO                  -->
+  <!-- ============================================== -->
+  <!-- Chassi principal -->
+  <link name="chassis_link">
+    <visual>
+      <geometry>
+        <box size="${chassis_length} ${chassis_width} ${chassis_height}"/>
+      </geometry>
+      <material name="grey">
+        <color rgba="0.5 0.5 0.5 1.0"/>
+      </material>
+    </visual>
+    <collision>
+      <geometry>
+        <box size="${chassis_length} ${chassis_width} ${chassis_height}"/>
+      </geometry>
+    </collision>
+  </link>
+  <!-- centro do chassi: o fundo do chassi fica (wheel_radius - wheel_projection) acima do base_link -->
+  <joint name="chassis_joint" type="fixed">
+    <parent link="base_link"/>
+    <child link="chassis_link"/>
+    <origin xyz="0 0 ${wheel_radius - wheel_projection + chassis_height/2.0}" rpy="0 0 0"/>
+  </joint>
+  <!-- Caixa do LiDAR no topo -->
+  <link name="lidar_box_link">
+    <visual>
+      <geometry>
+        <box size="${lidar_box_l} ${lidar_box_w} ${lidar_box_h}"/>
+      </geometry>
+      <material name="grey"/>
+    </visual>
+  </link>
+  <joint name="lidar_box_joint" type="fixed">
+    <parent link="chassis_link"/>
+    <child link="lidar_box_link"/>
+    <origin xyz="0 0 ${chassis_height/2.0 + lidar_box_h/2.0}" rpy="0 0 0"/>
+  </joint>
+  <!-- Pára-choque dianteiro -->
+  <link name="bumper_link">
+    <visual>
+      <geometry>
+        <box size="${bumper_length} ${bumper_width} ${bumper_height}"/>
+      </geometry>
+      <material name="dark_grey">
+        <color rgba="0.2 0.2 0.2 1.0"/>
+      </material>
+    </visual>
+    <collision>
+      <geometry>
+        <box size="${bumper_length} ${bumper_width} ${bumper_height}"/>
+      </geometry>
+    </collision>
+  </link>
+  <joint name="bumper_joint" type="fixed">
+    <parent link="base_link"/>
+    <child link="bumper_link"/>
+    <origin xyz="${chassis_length/2.0 + bumper_length/2.0} 0 ${wheel_radius - wheel_projection + bumper_height/2.0}" rpy="0 0 0"/>
+  </joint>
+  <!-- Pára-choque traseiro -->
+  <link name="rear_bumper_link">
+    <visual>
+      <geometry>
+        <box size="${bumper_length} ${bumper_width} ${bumper_height}"/>
+      </geometry>
+      <material name="dark_grey">
+        <color rgba="0.2 0.2 0.2 1.0"/>
+      </material>
+    </visual>
+    <collision>
+      <geometry>
+        <box size="${bumper_length} ${bumper_width} ${bumper_height}"/>
+      </geometry>
+    </collision>
+  </link>
+  <joint name="rear_bumper_joint" type="fixed">
+    <parent link="base_link"/>
+    <child link="rear_bumper_link"/>
+    <origin xyz="${-(chassis_length/2.0 + bumper_length/2.0)} 0 ${wheel_radius - wheel_projection + bumper_height/2.0}" rpy="0 0 0"/>
+  </joint>
+  <!-- Roda traseira esquerda (+Y) -->
+  <link name="rear_left_wheel_link">
+    <visual>
+      <geometry>
+        <cylinder radius="${wheel_radius}" length="${wheel_thickness}"/>
+      </geometry>
+      <material name="black">
+        <color rgba="0.1 0.1 0.1 1.0"/>
+      </material>
+    </visual>
+    <collision>
+      <geometry>
+        <cylinder radius="${wheel_radius}" length="${wheel_thickness}"/>
+      </geometry>
+    </collision>
+  </link>
+  <joint name="rear_left_wheel_joint" type="fixed">
+    <parent link="drive_wheel_link"/>
+    <child link="rear_left_wheel_link"/>
+    <origin xyz="0 ${half_track} 0" rpy="${-pi/2.0} 0 0"/>
+  </joint>
+  <!-- Roda traseira direita (−Y) -->
+  <link name="rear_right_wheel_link">
+    <visual>
+      <geometry>
+        <cylinder radius="${wheel_radius}" length="${wheel_thickness}"/>
+      </geometry>
+      <material name="black">
+        <color rgba="0.1 0.1 0.1 1.0"/>
+      </material>
+    </visual>
+    <collision>
+      <geometry>
+        <cylinder radius="${wheel_radius}" length="${wheel_thickness}"/>
+      </geometry>
+    </collision>
+  </link>
+  <joint name="rear_right_wheel_joint" type="fixed">
+    <parent link="drive_wheel_link"/>
+    <child link="rear_right_wheel_link"/>
+    <origin xyz="0 ${-half_track} 0" rpy="${-pi/2.0} 0 0"/>
+  </joint>
+  <!-- Roda dianteira esquerda (+Y) -->
+  <link name="front_left_wheel_link">
+    <visual>
+      <geometry>
+        <cylinder radius="${wheel_radius}" length="${wheel_thickness}"/>
+      </geometry>
+      <material name="black">
+        <color rgba="0.1 0.1 0.1 1.0"/>
+      </material>
+    </visual>
+    <collision>
+      <geometry>
+        <cylinder radius="${wheel_radius}" length="${wheel_thickness}"/>
+      </geometry>
+    </collision>
+  </link>
+  <joint name="front_left_wheel_joint" type="continuous">
+    <parent link="steering_link"/>
+    <child link="front_left_wheel_link"/>
+    <origin xyz="0 ${half_track} 0" rpy="${-pi/2.0} 0 0"/>
     <axis xyz="0 0 1"/>
-    <limit lower="${-max_steer_angle_right}" upper="${max_steer_angle_left}" effort="10.0" velocity="5.0"/>
-    <mimic joint="steering_joint" multiplier="1.0" offset="0.0"/>
-  </joint>
-  <link name="fl_wheel_link">
-    <visual>
-      <origin xyz="0 0 0" rpy="${pi/2} 0 0"/>
-      <geometry>
-        <cylinder radius="${wheel_radius}" length="${wheel_width}"/>
-      </geometry>
-      <material name="black"/>
-    </visual>
-  </link>
-  <joint name="fl_wheel_joint" type="continuous">
-    <parent link="fl_steer_link"/>
-    <child link="fl_wheel_link"/>
-    <origin xyz="0 0 0" rpy="0 0 0"/>
-    <axis xyz="0 1 0"/>
-    <mimic joint="drive_joint" multiplier="1.0" offset="0.0"/>
-  </joint>
-  <link name="fr_steer_link" />
-  <joint name="fr_steer_joint" type="revolute">
-    <parent link="base_link"/>
-    <child link="fr_steer_link"/>
-    <origin xyz="${wheelbase/2} ${-track_width/2} 0" rpy="0 0 0"/>
+  </joint>
+  <!-- Roda dianteira direita (−Y) -->
+  <link name="front_right_wheel_link">
+    <visual>
+      <geometry>
+        <cylinder radius="${wheel_radius}" length="${wheel_thickness}"/>
+      </geometry>
+      <material name="black">
+        <color rgba="0.1 0.1 0.1 1.0"/>
+      </material>
+    </visual>
+    <collision>
+      <geometry>
+        <cylinder radius="${wheel_radius}" length="${wheel_thickness}"/>
+      </geometry>
+    </collision>
+  </link>
+  <joint name="front_right_wheel_joint" type="continuous">
+    <parent link="steering_link"/>
+    <child link="front_right_wheel_link"/>
+    <origin xyz="0 ${-half_track} 0" rpy="${-pi/2.0} 0 0"/>
     <axis xyz="0 0 1"/>
-    <limit lower="${-max_steer_angle_right}" upper="${max_steer_angle_left}" effort="10.0" velocity="5.0"/>
-    <mimic joint="steering_joint" multiplier="1.0" offset="0.0"/>
-  </joint>
-  <link name="fr_wheel_link">
-    <visual>
-      <origin xyz="0 0 0" rpy="${pi/2} 0 0"/>
-      <geometry>
-        <cylinder radius="${wheel_radius}" length="${wheel_width}"/>
-      </geometry>
-      <material name="black"/>
-    </visual>
-  </link>
-  <joint name="fr_wheel_joint" type="continuous">
-    <parent link="fr_steer_link"/>
-    <child link="fr_wheel_link"/>
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